File: kicad/Arduino_Shield_RC_Controller/Arduino_Shield_RC_Controller.kicad_pcb (KiCad board)
At the start: 2 copper layers, 135 x 100 mm, 14 parts, among them SW1 PTS810SJG250SMTRLFS, SW2 PTS810SJG250SMTRLFS, SW3 PTS810SJG250SMTRLFS

Commit message: finished layout added a couple extra buttons
Parts:
- added SW4: PTS810SJG250SMTRLFS, Arduino_Shield_RC_Controller:PTS810, F.Cu at (155.7, 72.1)
- added SW5: PTS810SJG250SMTRLFS, Arduino_Shield_RC_Controller:PTS810, F.Cu at (165.1, 72.1)
- AR1: value (none) -> ARDUINO_R3
- J1: value (none) -> CONN_04X2
- LCD1: value (none) -> ADM1602K
- R1: value (none) -> R-TRIMM3103
- moved AR1 85.8 mm to (213.6, 57.4), turned to 180 degrees
- moved R5 56.2 mm to (154.7, 121.6), turned to 0 degrees
- moved LCD1 49.2 mm to (151.1, 134.1)
- moved R1 48.0 mm to (124.0, 109.0)
- moved J1 22.9 mm to (138.2, 61.5)
- moved C1 21.7 mm to (132.1, 61.6)
- moved C2 16.5 mm to (127.3, 58.9), turned to -90 degrees
- moved SW2 16.2 mm to (151.4, 92.7)
- moved @HOLE2 15.6 mm to (206.0, 59.4)
- moved SW1 14.8 mm to (98.8, 70.2)
- moved SW3 14.1 mm to (198.9, 70.9)
Connections:
- net MISO renamed /MISO
- net MOSI renamed /MOSI
- net SCK renamed Net-(AR1-SCK/PB5)
- net V0 renamed /V0
- AR1 pad P1: SCL -> unconnected-(AR1-SCL-PadP1)
- AR1 pad P10: D4 -> Net-(AR1-8)
- AR1 pad P11: D5 -> Net-(AR1-7)
- AR1 pad P12: CSN -> Net-(AR1-6)
- AR1 pad P13: SW3 -> Net-(AR1-5)
- AR1 pad P14: D6 -> Net-(AR1-4)
- AR1 pad P15: RCE -> Net-(AR1-3)
- AR1 pad P16: D7 -> Net-(AR1-2)
- AR1 pad P17: NC -> unconnected-(AR1-1-TX-PadP17)
- AR1 pad P18: NC -> unconnected-(AR1-0-RX-PadP18)
- AR1 pad P2: SDA -> unconnected-(AR1-SDA-PadP2)
- AR1 pad P20: VDD5 -> unconnected-(AR1-VDD5-PadP20)
- AR1 pad P23: N$9 -> unconnected-(AR1-RESET2-PadP23)
- AR1 pad P24: GND -> unconnected-(AR1-GND3-PadP24)
- AR1 pad P25: A5 -> Net-(AR1-A5)
- AR1 pad P26: A4 -> Net-(AR1-A4)
- AR1 pad P27: A3 -> Net-(AR1-A3)
- AR1 pad P28: A2 -> Net-(AR1-A2)
- AR1 pad P29: A1 -> unconnected-(AR1-A1-PadP29)
- AR1 pad P3: AREF -> unconnected-(AR1-AREF-PadP3)
- AR1 pad P30: A0 -> unconnected-(AR1-A0-PadP30)
- AR1 pad P31: VDD5 -> unconnected-(AR1-VIN-PadP31)
- AR1 pad P34: VDD5 -> +5V
- AR1 pad P35: VDD -> +3.3V
- AR1 pad P36: NC -> unconnected-(AR1-RESET-PadP36)
- AR1 pad P37: NC -> unconnected-(AR1-IOREF-PadP37)
- AR1 pad P38: NC -> unconnected-(AR1-NC-PadP38)
- AR1 pad P5: SW1 -> unconnected-(AR1-13-PadP5)
- AR1 pad P6: SW2 -> unconnected-(AR1-12-PadP6)
- AR1 pad P7: RS -> unconnected-(AR1-11-PadP7)
- AR1 pad P8: E -> Net-(AR1-10)
- AR1 pad P9: PWM9 -> Net-(AR1-9)
- C1 pad P$2: VDD -> +3.3V
- C2 pad 1: GND -> +3.3V
- C2 pad 2: VDD -> GND
- J1 pad 2: VDD -> +3.3V
- J1 pad 3: RCE -> Net-(AR1-A4)
- J1 pad 4: CSN -> Net-(AR1-A5)
- J1 pad 8: NC -> unconnected-(J1-Pad8)
- LCD1 pad P10: NC -> unconnected-(LCD1-DB3-PadP10)
- LCD1 pad P11: D4 -> Net-(AR1-4)
- LCD1 pad P12: D5 -> Net-(AR1-5)
- LCD1 pad P13: D6 -> Net-(AR1-6)
- LCD1 pad P14: D7 -> Net-(AR1-7)
- LCD1 pad P2: VDD5 -> +5V
- LCD1 pad P4: RS -> Net-(AR1-3)
- LCD1 pad P6: E -> Net-(AR1-2)
- LCD1 pad P7: NC -> unconnected-(LCD1-DB0-PadP7)
- LCD1 pad P8: NC -> unconnected-(LCD1-DB1-PadP8)
- LCD1 pad P9: NC -> unconnected-(LCD1-DB2-PadP9)
- R1 pad 1: VDD5 -> +5V
- R5 pad P$2: VDD5 -> +5V
- SW1 pad 1: SW1 -> Net-(AR1-8)
- SW1 pad 2: SW1 -> Net-(AR1-8)
- SW2 pad 1: SW2 -> Net-(AR1-9)
- SW2 pad 2: SW2 -> Net-(AR1-9)
- SW3 pad 1: SW3 -> Net-(AR1-10)
- SW3 pad 2: SW3 -> Net-(AR1-10)
Routing:
- net VDD5: track 324.1 -> 0.00 mm, vias 3 -> 0
- net VDD: track 118.6 -> 0.00 mm, vias 1 -> 0
- net Net-(AR1-8): track 0.00 -> 91.5 mm
- net SW1: track 82.2 -> 0.00 mm
- net RS: track 58.0 -> 0.00 mm, vias 1 -> 0
- net +3.3V: track 0.00 -> 55.2 mm
- net SW3: track 54.8 -> 0.00 mm
- net E: track 53.0 -> 0.00 mm, vias 1 -> 0
- net Net-(AR1-10): track 0.00 -> 52.5 mm
- net CSN: track 51.1 -> 0.00 mm
- net D4: track 41.0 -> 0.00 mm, vias 1 -> 0
- net Net-(AR1-3): track 0.00 -> 40.9 mm
- net D5: track 35.9 -> 0.00 mm, vias 1 -> 0
- net Net-(AR1-9): track 0.00 -> 32.1 mm
- net Net-(AR1-2): track 0.00 -> 31.8 mm
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- added copper zone on B.Cu, net +5V
- added copper zone on F.Cu, net +5V
- removed copper zone on F.Cu, net GND
Other:
- board text added: "1"
- board text added: "16"
- board text added: "2"
- board text added: "3.3V"
- board text added: "5V"
- board text added: "Analog In"
- board text added: "D0-7"
- board text added: "D8-13, GND, AREF, I2C"
- board text added: "G"
- board text added: "GND"
- board text added: "ICSP"
- board text added: "LCD"
- board text added: "Power"
- board text added: "nRF24L01"
