File: kicad/Arduino_Shield_RC_Controller/Arduino_Shield_RC_Controller.kicad_sch (KiCad schematic)
At the start: 10 parts, among them J1 CONN_04X2, SW1 PTS810SJG250SMTRLFS, SW2 PTS810SJG250SMTRLFS, SW3 PTS810SJG250SMTRLFS

Commit message: finished layout added a couple extra buttons
Parts:
- added SW4, SW5: PTS810SJG250SMTRLFS, Arduino_Shield_RC_Controller:PTS810, symbol Arduino_Shield_RC_Controller-eagle-import:PTS810SJG250SMTRLFS
Connections:
- net GND: now also C2.2, SW4.3, SW4.4, SW5.3, SW5.4; no longer AR1.P24 (GND3), C2.1
- net A0: no longer names the net of AR1.P30 (A0)
- net A1: no longer names the net of AR1.P29 (A1)
- net A2: no longer names the net of AR1.P28 (A2)
- net A2: now also SW5.1, SW5.2
- net A3: no longer names the net of AR1.P27 (A3)
- net A3: now also SW4.1, SW4.2
- net A4: no longer names the net of AR1.P26 (A4)
- net A4: now also J1.3
- net A5: no longer names the net of AR1.P25 (A5)
- net A5: now also J1.4
- net AREF: no longer names the net of AR1.P3 (AREF)
- net CSN: no longer names the net of AR1.P12 (6)
- net CSN: now also LCD1.P13 (DB6); no longer J1.4
- net D4: no longer names the net of LCD1.P11 (DB4)
- net D4: now also AR1.P14 (4); no longer AR1.P10 (8)
- net D5: no longer names the net of LCD1.P12 (DB5)
- net D5: now also AR1.P13 (5); no longer AR1.P11 (7)
- removed net D6: AR1.P14 (4), LCD1.P13 (DB6)
- net D7: no longer names the net of LCD1.P14 (DB7)
- net D7: now also AR1.P11 (7); no longer AR1.P16 (2)
- net E: no longer names the net of LCD1.P6 (E)
- net E: now also AR1.P16 (2); no longer AR1.P8 (10)
- net N$9: no longer names the net of AR1.P23 (RESET2)
- removed net NC: AR1.P17 (1-TX), AR1.P18 (0-RX), AR1.P36 (RESET), AR1.P37 (IOREF), AR1.P38 (NC), J1.8, LCD1.P10 (DB3), LCD1.P7 (DB0), LCD1.P8 (DB1), LCD1.P9 (DB2)
- net PWM9: no longer names the net of AR1.P9 (9)
- net PWM9: now also SW2.1, SW2.2
- net RCE: no longer names the net of AR1.P15 (3)
- net RCE: now also LCD1.P4 (RS); no longer J1.3
- net RS: no longer names the net of AR1.P7 (11)
- net RS: no longer LCD1.P4 (RS)
- net SCK: no longer names the net of AR1.P21 (SCK/PB5), J1.5
- net SCL: no longer names the net of AR1.P1 (SCL)
- net SDA: no longer names the net of AR1.P2 (SDA)
- net SW1: no longer names the net of SW1.1, SW1.2
- net SW1: now also AR1.P10 (8); no longer AR1.P5 (13)
- removed net SW2: AR1.P6 (12), SW2.1, SW2.2
- net SW3: no longer names the net of SW3.1, SW3.2
- net SW3: now also AR1.P8 (10); no longer AR1.P13 (5)
- net VDD renamed +3.3V
- net +3.3V: now also C2.1; no longer C2.2
- net VDD5 renamed +5V
- net +5V: no longer AR1.P20 (VDD5), AR1.P31 (VIN)
- no-connect marks 0 -> 20
Other:
- moved on the sheet: C1
