File: kicad/ArduinoShieldServoMotors/ArduinoShieldServoMotors.kicad_pcb (KiCad board)
At the start: 2 copper layers, 68.6 x 53.3 mm, 15 parts, among them J1 Power, J10 Conn_01x03, J12 Screw_Terminal_01x02, J2 Digital/PWM, J3 Analog, J4 Digital/PWM, J5 Conn_01x03, J6 Conn_01x03, J7 Conn_01x03, J8 Conn_01x03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

Commit message: sent off ArduinoShieldServoMotors to JLCPCB
Parts:
- added C1: 470 ufd, Capacitor_THT:CP_Radial_D10.0mm_P5.00mm, F.Cu at (160.0, 71.6)
- added D7: Conn_01x03, Connector_PinHeader_2.54mm:PinHeader_1x03_P2.54mm_Vertical, F.Cu at (146.5, 61.6)
- added D8: Conn_01x03, Connector_PinHeader_2.54mm:PinHeader_1x03_P2.54mm_Vertical, F.Cu at (146.5, 56.6)
- +__5V__-1: renamed from J12; footprint TerminalBlock:TerminalBlock_bornier-3_P5.08mm -> TerminalBlock:TerminalBlock_bornier-2_P5.08mm
- moved A0 25.8 mm to (146.5, 92.1), turned to -90 degrees
- moved A1 18.9 mm to (146.5, 87.0), turned to -90 degrees
- moved +__5V__-1 18.5 mm to (158.4, 61.4), turned to 90 degrees
- moved A2 12.0 mm to (146.5, 82.0), turned to -90 degrees
- moved D4 8.63 mm to (146.5, 66.7), turned to -90 degrees
- moved A3 5.15 mm to (146.5, 76.9), turned to -90 degrees
- moved D2 1.74 mm to (146.5, 71.8), turned to -90 degrees
- renumbered J5 to A0, J6 to A1, J7 to A2, J8 to A3, J9 to D2, J10 to D4
Connections:
- A0 pad 1: /SCL/A5 -> /A0
- A1 pad 1: /SDA/A4 -> /A1
- A2 pad 1: /A3 -> /A2
- A3 pad 1: /A2 -> /A3
- D2 pad 1: /A1 -> /2
- D4 pad 1: /A0 -> /4
- J1 pad 1: unconnected-(J1-Pin_1-Pad1) -> /AREF
Routing:
- net GND: track 0.00 -> 102.5 mm
- net Net-(+__5V__-1-Pin_1): track 0.00 -> 64.0 mm
- net /2: track 0.00 -> 28.7 mm
- net /A3: track 0.00 -> 25.5 mm
- net /4: track 0.00 -> 20.4 mm
- net /A2: track 0.00 -> 19.4 mm
- net /7: track 0.00 -> 14.7 mm
- net /A1: track 0.00 -> 13.3 mm
- net /8: track 0.00 -> 11.4 mm
- net /A0: track 0.00 -> 7.12 mm
Other:
- board text added: "+ 5V -"
- board text added: "5V"
- board text added: "GND"
- board text removed: "ICSP"
