File: kicad/ArduinoShieldServoMotors/ArduinoShieldServoMotors.kicad_sch (KiCad schematic)
At the start: 11 parts, among them J1 Power, J10 Conn_01x03, J12 Screw_Terminal_01x02, J2 Digital/PWM, J3 Analog, J4 Digital/PWM, J5 Conn_01x03, J6 Conn_01x03, J7 Conn_01x03, J8 Conn_01x03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

Commit message: sent off ArduinoShieldServoMotors to JLCPCB
Parts:
- added C1: 470 ufd, Capacitor_THT:CP_Radial_D10.0mm_P5.00mm, symbol Device:C_Polarized
- added D7, D8: Conn_01x03, Connector_PinHeader_2.54mm:PinHeader_1x03_P2.54mm_Vertical, symbol Connector_Generic:Conn_01x03
- +__5V__-1: renamed from J12; footprint TerminalBlock:TerminalBlock_bornier-3_P5.08mm -> TerminalBlock:TerminalBlock_bornier-2_P5.08mm
- renumbered J5 to A0, J6 to A1, J7 to A2, J8 to A3, J9 to D2, J10 to D4
Connections:
- net 2: now also D2.1 (Pin_1)
- net 4: now also D4.1 (Pin_1)
- net 7: now also D7.1 (Pin_1)
- net 8: now also D8.1 (Pin_1)
- net A0: now also A0.1 (Pin_1); no longer D4.1 (Pin_1)
- net A1: now also A1.1 (Pin_1); no longer D2.1 (Pin_1)
- net A2: now also A2.1 (Pin_1); no longer A3.1 (Pin_1)
- net A3: now also A3.1 (Pin_1); no longer A2.1 (Pin_1)
- net AREF: now also J1.1 (Pin_1)
- net GND: now also C1.2, D7.3 (Pin_3), D8.3 (Pin_3)
- net SCL/A5: no longer A0.1 (Pin_1)
- net SDA/A4: no longer A1.1 (Pin_1)
- net at +__5V__-1.1 (Pin_1), A0.2 (Pin_2), A1.2 (Pin_2)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: now also C1.1, D7.2 (Pin_2), D8.2 (Pin_2)
Other:
- moved on the sheet: D2, D4
