File: kicad/nRF_servo_Mega/nRF_servo_Mega.kicad_pcb (KiCad board)
At the start: 2 copper layers, 85.1 x 53.3 mm, 12 parts, among them J1 Screw_Terminal_01x02, M3 Motor_Servo, U1 NRF24L01_Breakout

Commit message: added servo pinouts to silkscreen
Other:
- board text added: "S"
- board text removed: "P"
Changed lines of the file:
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@@
 		(tags "Through hole pin header THT 1x03 2.54mm single row")
 		(property "Reference" "D21"
-			(at 0 -2.794 270)
+			(at 0 -2.794 -90)
 			(layer "B.SilkS")
 			(effects
@@
 			(at -1.778 4.826 -90)
 			(layer "B.SilkS")
+			(hide yes)
 			(effects
 				(font
@@
 			(at -2.54 -0.762 180)
 			(layer "B.SilkS")
+			(hide yes)
 			(effects
 				(font
@@
 		(tags "CP Radial series Radial pin pitch 5.00mm  diameter 10mm Electrolytic Capacitor")
 		(property "Reference" "C2"
-			(at 3.048 -6.604 0)
+			(at 8.652 -4.462 0)
 			(layer "B.SilkS")
 			(effects
@@
 		)
 		(property "Value" "470 uF"
-			(at 1.524 -8.128 0)
+			(at 7.152 -5.962 0)
 			(layer "B.SilkS")
 			(effects
@@
 	)
 	(gr_text "GND"
-		(at 36.322 47.752 -90)
+		(at 35.5 49 270)
 		(layer "B.SilkS")
 		(effects
 			(font
-				(size 1 1)
-				(thickness 0.15)
+				(size 1.5 1.5)
+				(thickness 0.2)
 			)
 			(justify left bottom mirror)
@@
 		)
 	)
-	(gr_text "P"
+	(gr_text "S"
 		(at 49.5 24 270)
 		(layer "B.SilkS")
@@
 		)
 	)
-	(gr_text "P"
+	(gr_text "S"
 		(at 38 24 270)
 		(layer "B.SilkS")
@@
 		)
 	)
-	(gr_text "P"
+	(gr_text "S"
 		(at 49.5 34 270)
 		(layer "B.SilkS")
@@
 		)
 	)
-	(gr_text "P"
+	(gr_text "S"
 		(at 38 29 270)
 		(layer "B.SilkS")
@@
 	)
 	(gr_text "+5V"
-		(at 36.322 43.688 -90)
+		(at 35.5 43.5 270)
 		(layer "B.SilkS")
 		(effects
 			(font
-				(size 1 1)
-				(thickness 0.15)
+				(size 1.5 1.5)
+				(thickness 0.2)
 			)
 			(justify left bottom mirror)
@@
 		)
 	)
-	(gr_text "P"
+	(gr_text "S"
 		(at 49.5 29 270)
 		(layer "B.SilkS")
@@
 		)
 	)
-	(gr_text "P"
+	(gr_text "S"
 		(at 38 34 270)
 		(layer "B.SilkS")
@@
 	)
 	(gr_text_box "nRF Servo Mega\nMichael Shiloh 2024, 2025\nGPLv3 Applies\n\nRevision 0.2 Sept 2025\n"
-		(start 72.192 34.29)
-		(end 106.426 48.808)
+		(start 75.5 39.5)
+		(end 109.734 54.018)
+		(layer "B.SilkS")
+		(effects
+			(font
+				(size 1.5 1.5)
+				(thickness 0.2)
+			)
+			(justify left top mirror)
+		)
+		(border yes)
+		(stroke
+			(width 0.2)
+			(type solid)
+		)
+	)
+	(gr_text_box "Pin order for all \nsix sets of 3 pins\n\nGND  +5V  Signal\n"
+		(start 35.0025 21.741)
+		(end 91.234 38.259)
 		(layer "B.SilkS")
 		(effects
 			(font
 				(size 1.5 1.5)
-				(thickness 0.3)
-				(bold yes)
+				(thickness 0.2)
 			)
 			(justify left top mirror)
