File: kicad/arduinoMegaServoShield/arduinoMegaServoShield.kicad_pcb (KiCad board)
At the start: 2 copper layers, 101.6 x 53.4 mm, 39 parts, among them J1 Screw_Terminal_01x02, M1 Motor_Servo, M10 Motor_Servo, M11 Motor_Servo, M12 Motor_Servo, M13 Motor_Servo, M14 Motor_Servo, M15 Motor_Servo, M16 Motor_Servo, M17 Motor_Servo, M18 Motor_Servo, M19 Motor_Servo, M2 Motor_Servo, M20 Motor_Servo, M21 Motor_Servo, M23 Motor_Servo, M25 Motor_Servo, M26 Motor_Servo, M27 Motor_Servo, M28 Motor_Servo, M29 Motor_Servo, M30 Motor_Servo, M31 Motor_Servo, M34 Motor_Servo, M35 Motor_Servo, M36 Motor_Servo, M37 Motor_Servo, M38 Motor_Servo, M39 Motor_Servo, M4 Motor_Servo, M40 Motor_Servo, M41 Motor_Servo, M5 Motor_Servo, M6 Motor_Servo, M7 Motor_Servo, M8 Motor_Servo, M9 Motor_Servo

Commit message: minor changes for Machine Lab 2026
Parts:
- removed M39, M41: Motor_Servo, Connector_PinHeader_2.54mm:PinHeader_1x03_P2.54mm_Vertical
- added M3: Motor_Servo, Connector_PinHeader_2.54mm:PinHeader_1x03_P2.54mm_Vertical, F.Cu at (39.9, 34.5)
- moved M15 59.4 mm to (107.7, 33.0)
- moved M30 25.1 mm to (52.3, 55.9)
Connections:
- M1 pad 2: unconnected-(M1-+-Pad2) -> +5VP
- M1 pad 3: unconnected-(M1---Pad3) -> GND
- M10 pad 2: unconnected-(M10-+-Pad2) -> +5VP
- M10 pad 3: unconnected-(M10---Pad3) -> GND
- M11 pad 2: unconnected-(M11-+-Pad2) -> +5VP
- M11 pad 3: unconnected-(M11---Pad3) -> GND
- M12 pad 2: unconnected-(M12-+-Pad2) -> +5VP
- M12 pad 3: unconnected-(M12---Pad3) -> GND
- M13 pad 2: unconnected-(M13-+-Pad2) -> +5VP
- M13 pad 3: unconnected-(M13---Pad3) -> GND
- M14 pad 2: unconnected-(M14-+-Pad2) -> +5VP
- M14 pad 3: unconnected-(M14---Pad3) -> GND
- M15 pad 1: unconnected-(M15-PWM-Pad1) -> Net-(M15-PWM)
- M15 pad 2: unconnected-(M15-+-Pad2) -> +5VP
- M15 pad 3: unconnected-(M15---Pad3) -> GND
- M16 pad 2: unconnected-(M16-+-Pad2) -> +5VP
- M16 pad 3: unconnected-(M16---Pad3) -> GND
- M17 pad 2: unconnected-(M17-+-Pad2) -> +5VP
- M17 pad 3: unconnected-(M17---Pad3) -> GND
- M18 pad 2: unconnected-(M18-+-Pad2) -> +5VP
- M18 pad 3: unconnected-(M18---Pad3) -> GND
- M19 pad 2: unconnected-(M19-+-Pad2) -> +5VP
- M19 pad 3: unconnected-(M19---Pad3) -> GND
- M20 pad 1: unconnected-(M20-PWM-Pad1) -> Net-(M20-PWM)
- M20 pad 2: unconnected-(M20-+-Pad2) -> +5VP
- M20 pad 3: unconnected-(M20---Pad3) -> GND
- M21 pad 1: unconnected-(M21-PWM-Pad1) -> Net-(M21-PWM)
- M21 pad 2: unconnected-(M21-+-Pad2) -> +5VP
- M21 pad 3: unconnected-(M21---Pad3) -> GND
- M23 pad 2: unconnected-(M23-+-Pad2) -> +5VP
- M23 pad 3: unconnected-(M23---Pad3) -> GND
- M25 pad 1: unconnected-(M25-PWM-Pad1) -> Net-(M25-PWM)
- M25 pad 2: unconnected-(M25-+-Pad2) -> +5VP
- M25 pad 3: unconnected-(M25---Pad3) -> GND
- M26 pad 1: unconnected-(M26-PWM-Pad1) -> Net-(M26-PWM)
- M26 pad 2: unconnected-(M26-+-Pad2) -> +5VP
- M26 pad 3: unconnected-(M26---Pad3) -> GND
- M27 pad 2: unconnected-(M27-+-Pad2) -> +5VP
- M27 pad 3: unconnected-(M27---Pad3) -> GND
- M28 pad 2: unconnected-(M28-+-Pad2) -> +5VP
- M28 pad 3: unconnected-(M28---Pad3) -> GND
- M29 pad 2: unconnected-(M29-+-Pad2) -> +5VP
- M29 pad 3: unconnected-(M29---Pad3) -> GND
- M30 pad 2: unconnected-(M30-+-Pad2) -> +5VP
- M30 pad 3: unconnected-(M30---Pad3) -> GND
- M31 pad 2: unconnected-(M31-+-Pad2) -> +5VP
- M31 pad 3: unconnected-(M31---Pad3) -> GND
- M34 pad 2: unconnected-(M34-+-Pad2) -> +5VP
- M34 pad 3: unconnected-(M34---Pad3) -> GND
- M35 pad 2: unconnected-(M35-+-Pad2) -> +5VP
- M35 pad 3: unconnected-(M35---Pad3) -> GND
- M36 pad 2: unconnected-(M36-+-Pad2) -> +5VP
- M36 pad 3: unconnected-(M36---Pad3) -> GND
- M37 pad 2: unconnected-(M37-+-Pad2) -> +5VP
- M37 pad 3: unconnected-(M37---Pad3) -> GND
- M38 pad 2: unconnected-(M38-+-Pad2) -> +5VP
- M38 pad 3: unconnected-(M38---Pad3) -> GND
- M40 pad 2: unconnected-(M40-+-Pad2) -> +5VP
- M40 pad 3: unconnected-(M40---Pad3) -> GND
- M5 pad 1: Net-(M5-PWM) -> +5VP
- M5 pad 2: unconnected-(M5-+-Pad2) -> +5VP
- M5 pad 3: unconnected-(M5---Pad3) -> GND
- M6 pad 2: unconnected-(M6-+-Pad2) -> +5VP
- M6 pad 3: unconnected-(M6---Pad3) -> GND
- M7 pad 2: unconnected-(M7-+-Pad2) -> +5VP
- M7 pad 3: unconnected-(M7---Pad3) -> GND
- M8 pad 2: unconnected-(M8-+-Pad2) -> +5VP
- M8 pad 3: unconnected-(M8---Pad3) -> GND
- M9 pad 2: unconnected-(M9-+-Pad2) -> +5VP
- M9 pad 3: unconnected-(M9---Pad3) -> GND
- XA1 pad A10: Net-(M14-PWM) -> Net-(M34-PWM)
- XA1 pad A11: unconnected-(XA1-PadA11) -> Net-(M13-PWM)
- XA1 pad A15: Net-(M5-PWM) -> +5VP
- XA1 pad A3: Net-(M28-PWM) -> Net-(M20-PWM)
- XA1 pad A4: unconnected-(XA1-PadA4) -> Net-(M21-PWM)
- XA1 pad A5: Net-(M23-PWM) -> Net-(M9-PWM)
- XA1 pad A6: Net-(M9-PWM) -> Net-(M16-PWM)
- XA1 pad A8: Net-(M34-PWM) -> Net-(M14-PWM)
- XA1 pad A9: Net-(M13-PWM) -> Net-(M30-PWM)
- XA1 pad D12: unconnected-(XA1-PadD12) -> Net-(M15-PWM)
- XA1 pad D14: unconnected-(XA1-D14/TX3-PadD14) -> Net-(M11-PWM)
- XA1 pad D15: unconnected-(XA1-D15/RX3-PadD15) -> Net-(M12-PWM)
- XA1 pad D16: unconnected-(XA1-D16/TX2-PadD16) -> Net-(M6-PWM)
- XA1 pad D17: unconnected-(XA1-D17/RX2-PadD17) -> Net-(M7-PWM)
- XA1 pad D21: Net-(M11-PWM) -> unconnected-(XA1-D21/SCL-PadD21)
- XA1 pad D24: Net-(M6-PWM) -> unconnected-(XA1-PadD24)
- XA1 pad D3: unconnected-(XA1-D3_INT1-PadD3) -> Net-(M23-PWM)
- XA1 pad D30: Net-(M12-PWM) -> unconnected-(XA1-PadD30)
- XA1 pad D32: Net-(M7-PWM) -> Net-(M3-PWM)
- XA1 pad D34: Net-(M30-PWM) -> Net-(M28-PWM)
- XA1 pad D36: Net-(M16-PWM) -> Net-(M31-PWM)
- XA1 pad D38: Net-(M31-PWM) -> Net-(M8-PWM)
- XA1 pad D4: unconnected-(XA1-PadD4) -> Net-(M25-PWM)
- XA1 pad D40: Net-(M8-PWM) -> unconnected-(XA1-PadD40)
- XA1 pad D42: unconnected-(XA1-PadD42) -> Net-(M2-PWM)
- XA1 pad D46: Net-(M2-PWM) -> unconnected-(XA1-PadD46)
- XA1 pad D5: unconnected-(XA1-PadD5) -> Net-(M26-PWM)
- XA1 pad GND4: unconnected-(XA1-SPI_GND-PadGND4) -> GND
Routing:
- net Net-(M28-PWM): track 0.00 -> 38.6 mm
- net GND: track 0.00 -> 37.5 mm
- net Net-(M16-PWM): track 0.00 -> 35.6 mm
- net Net-(M34-PWM): track 0.00 -> 35.5 mm
- net Net-(M21-PWM): track 0.00 -> 24.5 mm
- net Net-(M23-PWM): track 0.00 -> 24.0 mm
- net Net-(M13-PWM): track 0.00 -> 22.4 mm
- net Net-(M11-PWM): track 32.0 -> 11.6 mm
- net Net-(M15-PWM): track 0.00 -> 18.4 mm
- net Net-(M12-PWM): track 36.1 -> 19.6 mm
- net Net-(M25-PWM): track 0.00 -> 15.8 mm
- net Net-(M6-PWM): track 22.4 -> 7.37 mm
- net Net-(M20-PWM): track 0.00 -> 13.9 mm
- net Net-(M26-PWM): track 0.00 -> 10.3 mm
- net Net-(M5-PWM): track 7.93 -> 0.00 mm
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Other:
- board size 101.6 x 53.4 mm -> 101.6 x 53.3 mm
- board text added: "A0"
- board text added: "A1"
- board text added: "A10"
- board text added: "A11"
- board text added: "A15"
- board text added: "A2"
- board text added: "A3"
- board text added: "A4"
- board text added: "A5"
- board text added: "A6"
- board text added: "A7"
- board text added: "A8"
- board text added: "A9"
- board text added: "D10"
- board text added: "D11"
- board text added: "D12"
- board text added: "D13"
- board text added: "D14"
- board text added: "D15"
- board text added: "D16"
- board text added: "D17"
- board text added: "D22"
- board text added: "D3"
- board text added: "D32"
- board text added: "D34"
- board text added: "D36"
- board text added: "D38"
- board text added: "D4"
- board text added: "D42"
- board text added: "D48"
- board text added: "D5"
- board text added: "D6"
- board text added: "D7"
- board text added: "D8"
- board text added: "D9"
