File: kicad/motorMatrixAdapter/motorMatrixAdapter.kicad_pcb (KiCad board)
At the start: 2 copper layers, 2 parts

Commit message: soldering
Parts:
- moved REF** 0.18 mm to (106.7, 56.0)
Routing:
- net (no net): track 19.6 -> 71.3 mm
- added copper zone on F.Cu, net (none)
Other:
- board outline added: 13.2 x 16.3 mm
- board text added: "GND"
