File: kicad/mega_nRF_feedthrough/mega_nRF_feedthrough.kicad_pcb (KiCad board)
At the start: 2 copper layers, 102.1 x 53.2 mm, 11 parts, among them J1 Conn_01x08_Pin, J2 Conn_01x08_Pin, J3 Conn_01x10_Pin, J4 Conn_01x08_Pin, J6 Conn_01x08_Pin, J7 Conn_01x36, J8 Conn_01x06, U1 NRF24L01_Breakout, U2 AP2127N-3.3

Commit message: done
Parts:
- removed J1, J2, J4, J6: Conn_01x08_Pin, Connector_PinHeader_2.54mm:PinHeader_1x08_P2.54mm_Vertical
- removed J3: Conn_01x10_Pin, Connector_PinHeader_2.54mm:PinHeader_1x10_P2.54mm_Vertical
- removed J7: Conn_01x36, Connector_PinHeader_2.54mm:PinHeader_2x18_P2.54mm_Vertical
- removed J8: Conn_01x06, Connector_PinHeader_2.54mm:PinHeader_2x03_P2.54mm_Vertical
- added A1: Arduino_Mega2560_R3_Shield, PCM_arduino-library:Arduino_Mega2560_R3_Shield, F.Cu at (164.3, 90.9)
- added C3: 470uF, Capacitor_THT:CP_Radial_D8.0mm_P3.50mm, F.Cu at (251.7, 71.9)
- added C4: 3.3 uf, Capacitor_Tantalum_SMD:CP_EIA-3216-18_Kemet-A, F.Cu at (252.2, 78.0)
- C1, C2, U1, U2: moved to F.Cu
- moved C2 219.9 mm to (252.2, 84.1), turned to 0 degrees
- moved U2 215.4 mm to (250.7, 82.6), turned to -90 degrees
- moved C1 210.0 mm to (248.2, 81.0), turned to 180 degrees
- moved U1 209.7 mm to (249.7, 76.5)
Connections:
- net /5V renamed +5V
- net /GND renamed GND
- U1 pad 3: /D50 -> Net-(A1-D50_MISO)
- U1 pad 4: /D52 -> Net-(A1-D52_SCK)
- U1 pad 5: /SCK -> Net-(A1-SPI_SCK)
- U1 pad 6: /MOSI -> Net-(A1-SPI_MOSI)
- U1 pad 7: /MISO -> Net-(A1-SPI_MISO)
Routing:
- net /MISO: track 40.1 -> 0.00 mm
- net /MOSI: track 37.6 -> 0.00 mm
- net /SCK: track 37.4 -> 0.00 mm
- net Net-(A1-SPI_MISO): track 0.00 -> 33.9 mm
- net Net-(A1-SPI_MOSI): track 0.00 -> 31.0 mm
- net Net-(A1-SPI_SCK): track 0.00 -> 30.2 mm
- net /D52: track 16.0 -> 0.00 mm
- net Net-(A1-D50_MISO): track 0.00 -> 14.1 mm
- net /D50: track 13.0 -> 0.00 mm
- net Net-(A1-D52_SCK): track 0.00 -> 12.7 mm
- net Net-(U1-VCC): track 5.66 -> 14.1 mm
- added copper zone on B.Cu, net +5V
- added copper zone on F.Cu, net GND
- removed copper zone on F.Cu, net +5V
- removed copper zone on B.Cu, net GND
Other:
- board size 102.1 x 53.2 mm -> 99.3 x 53.6 mm
