File: kicad/mega_nRF_feedthrough/mega_nRF_feedthrough.kicad_pcb (KiCad board)
At the start: 2 copper layers, 99.3 x 53.6 mm, 7 parts, among them U1 NRF24L01_Breakout, U2 AP2127N-3.3

Commit message: added readme
Parts:
- C1, C2: footprint Capacitor_SMD:C_0201_0603Metric -> Capacitor_SMD:C_0603_1608Metric
- C4: footprint Capacitor_Tantalum_SMD:CP_EIA-3216-18_Kemet-A -> Capacitor_Tantalum_SMD:CP_EIA-3216-18_Kemet-A_HandSolder
- moved C2 0.40 mm to (252.5, 84.3)
Connections:
- A1 pad D46: unconnected-(A1-PadD46) -> Net-(U1-CE)
- A1 pad D48: unconnected-(A1-PadD48) -> Net-(U1-~{CSN})
- A1 pad D50: Net-(A1-D50_MISO) -> unconnected-(A1-D50_MISO-PadD50)
- A1 pad D52: Net-(A1-D52_SCK) -> unconnected-(A1-D52_SCK-PadD52)
- U1 pad 3: Net-(A1-D50_MISO) -> Net-(U1-CE)
- U1 pad 4: Net-(A1-D52_SCK) -> Net-(U1-~{CSN})
Routing:
- net Net-(U1-~{CSN}): track 0.00 -> 14.6 mm
- net Net-(A1-D50_MISO): track 14.1 -> 0.00 mm
- net Net-(U1-CE): track 0.00 -> 13.3 mm
- net Net-(A1-D52_SCK): track 12.7 -> 0.00 mm
- net Net-(A1-SPI_MOSI): track 31.0 -> 23.0 mm
- net Net-(A1-SPI_MISO): track 33.9 -> 26.8 mm
- net Net-(A1-SPI_SCK): track 30.2 -> 23.5 mm
